Commit message: Add PID controller

File: launch_pad.urdf (robot description, URDF)
Before this commit: robot launch_pad, 1 links, 0 joints
Links:
- link base_link: mass None -> 10; geometry collision box size=2 2 0.2; visual box size=2 2 0.2

Commit message: updated_new_reward_function

File: launch_pad.urdf (robot description, URDF)
Before this commit: robot launch_pad.urdf, 1 links, 0 joints
Links:
- link base_link: geometry collision box size=0.5 0.5 0.1; visual box size=0.5 0.5 0.1
