Commit message: Add wind effect and obstacles

File: box.urdf (robot description, URDF)
Before this commit: robot test.urdf, 1 links, 0 joints
Links:
- link baseLink: geometry collision box size=0.5 0.5 0.5; visual box size=0.5 0.5 0.5

File: launch_pad.urdf (robot description, URDF)
Before this commit: robot launch_pad.urdf, 1 links, 0 joints
Links:
- link base_link: geometry collision box size=0.5 0.5 0.1; visual box size=0.5 0.5 0.1

File: racer.urdf (robot description, URDF)
Before this commit: robot cf2, 6 links, 5 joints
Links:
- link base_link: mass 0.027 -> 0.830; geometry collision cylinder length=.025 radius=.06; visual mesh filename=./cf2.dae scale=3 3 3
